Commit message: Step5.1-inertial param

File: urdf/rebot.urdf (robot description, URDF)
Before this commit: robot rebot, 7 links, 6 joints
Links:
- link base_link: mass None -> 3.0; geometry collision box size=0.7 0.7 0.3; visual box size=0.7 0.7 0.3
- link left_finger: mass None -> 0.05; geometry collision box size=0.02 0.02 0.1; visual box size=0.02 0.02 0.1
- link link2: mass None -> 1.5; geometry collision box size=0.4 0.4 0.7; visual box size=0.4 0.4 0.7
- link link3: mass None -> 0.3; geometry collision cylinder length=0.25 radius=0.04; visual cylinder length=0.25 radius=0.04
- link link4: mass None -> 0.2; geometry collision cylinder length=0.2 radius=0.035; visual cylinder length=0.2 radius=0.035
- link link5: mass None -> 0.1; geometry collision cylinder length=0.15 radius=0.03; visual cylinder length=0.15 radius=0.03
- link right_finger: mass None -> 0.05; geometry collision box size=0.02 0.02 0.1; visual box size=0.02 0.02 0.1
